File: i2cmd.kicad_pcb (KiCad board)
At the start: 2 copper layers, 16 parts, among them CON1 BARREL_JACK, P1 CONN_02X03, P2 CONN_02X03, P3 CONN_02X03, P4 CONN_02X03, P5 CONN_02X03, P6 CONN_02X03, SW1 Switch_DPST, SW2 CONN_01X02, U1 NTC_C.H.I.P

Commit message: Improvements on the silkscreen.
Parts:
- turned JP1 to 180 degrees
- turned JP2 to 180 degrees
Routing:
- added copper zone on F.Cu, net +5V
- added copper zone on B.Cu, net GND
